Commit message: Fixed OakD URDF (#99)

File: clearpath_sensors_description/urdf/luxonis_oakd.urdf.xacro (robot description, xacro)
@@ -1,5 +1,19 @@
 <?xml version="1.0"?>
 <robot xmlns:xacro="http://ros.org/wiki/xacro">
+<xacro:macro name="inertial_dummy">
+  <xacro:property name="mass" value="0.01"/>
+  <xacro:property name="x" value="0.01"/>
+  <xacro:property name="y" value="0.01"/>
+  <xacro:property name="z" value="0.01"/>
+  <inertial>
+    <mass value="${mass}" />
+    <origin xyz="0 0 0" />
+    <inertia ixx="${(1/12) * mass * (y*y + z*z)}" ixy="0.0" ixz="0.0"
+      iyy="${(1/12) * mass * (x*x + z*z)}" iyz="0.0"
+      izz="${(1/12) * mass * (x*x + y*y)}" />
+  </inertial>
+</xacro:macro>
 <xacro:macro name="luxonis_oakd" params="name parent_link *origin model:=pro">
+  <xacro:property name="cm2m" value="0.01"/>
   <xacro:property name="mass"       value="0.061"/>
   <xacro:property name="baseline" value="0.075" />
@@ -21,5 +35,5 @@
     <visual>
       <geometry>
-        <mesh filename="package://clearpath_sensors_description/meshes/${name}_${model}.dae" scale="1 1 1" />
+        <mesh filename="package://clearpath_sensors_description/meshes/oakd_${model}.dae" scale="1 1 1" />
       </geometry>
     </visual>
@@ -115,5 +129,5 @@
       <visualize>true</visualize>
     </sensor>
-    <xacro:material_darkgray/>
+    <material name="clearpath_dark_grey"/>
   </gazebo>
   <gazebo reference="${name}_joint">
