Commit message: Add PTZ sim support (#125)
* Now that axis_camera is released via OSRF, depend on the official package, remove duplicate meshes

* Rename Gazebo plugins for Jazzy compatibility

* Modify Axis camera URDFs to using the axis_camera meshes. This lets us control the gazebo topics. Fix the GZ topic names. Camera data is now visible in the simulation

* Add joint controllers for the pan & tilt actuators. This provides velocity control over the simulated camera

File: clearpath_manipulators_description/urdf/arm/kinova_gen3_6dof.urdf.xacro (robot description, xacro)
@@ -362,5 +362,5 @@
           </xacro:if>
           <xacro:if value="${sim_ignition}">
-            <plugin>gz_ros2_control/IgnitionSystem</plugin>
+            <plugin>gz_ros2_control/GazeboSimSystem</plugin>
           </xacro:if>
           <xacro:if value="${sim_isaac}">

File: clearpath_manipulators_description/urdf/arm/kinova_gen3_7dof.urdf.xacro (robot description, xacro)
@@ -477,5 +477,5 @@
           </xacro:if>
           <xacro:if value="${sim_ignition}">
-            <plugin>gz_ros2_control/IgnitionSystem</plugin>
+            <plugin>gz_ros2_control/GazeboSimSystem</plugin>
           </xacro:if>
           <xacro:if value="${sim_isaac}">

File: clearpath_manipulators_description/urdf/arm/kinova_gen3_lite.urdf.xacro (robot description, xacro)
@@ -243,5 +243,5 @@
           </xacro:if>
           <xacro:if value="${sim_ignition}">
-            <plugin>gz_ros2_control/IgnitionSystem</plugin>
+            <plugin>gz_ros2_control/GazeboSimSystem</plugin>
           </xacro:if>
           <xacro:if value="${sim_isaac}">

File: clearpath_manipulators_description/urdf/gripper/kinova_2f_lite.urdf.xacro (robot description, xacro)
@@ -196,5 +196,5 @@
             </xacro:if>
               <xacro:if value="${sim_ignition}">
-                  <plugin>gz_ros2_control/IgnitionSystem</plugin>
+                  <plugin>gz_ros2_control/GazeboSimSystem</plugin>
               </xacro:if>
               <xacro:if value="${use_fake_hardware}">

File: clearpath_manipulators_description/urdf/gripper/robotiq_2f_140.urdf.xacro (robot description, xacro)
@@ -283,5 +283,5 @@
           </xacro:if>
           <xacro:if value="${sim_gazebo}">
-            <plugin>gz_ros2_control/IgnitionSystem</plugin>
+            <plugin>gz_ros2_control/GazeboSimSystem</plugin>
           </xacro:if>
           <xacro:if value="${use_fake_hardware}">

File: clearpath_platform_description/urdf/a300/mobility/diff_drive.urdf.xacro (robot description, xacro)
@@ -63,5 +63,5 @@
         <hardware>
           <xacro:if value="$(arg is_sim)">
-            <plugin>ign_ros2_control/IgnitionSystem</plugin>
+            <plugin>gz_ros2_control/GazeboSimSystem</plugin>
           </xacro:if>
           <xacro:unless value="$(arg is_sim)">

File: clearpath_sensors_description/urdf/axis/axis_dome_fixed.urdf.xacro (robot description, xacro)
@@ -13,5 +13,5 @@
       <visual>
         <geometry>
-          <mesh filename="package://clearpath_sensors_description/meshes/axis_dome.stl" scale="1 1 1" />
+          <mesh filename="package://axis_description/meshes/axis_dome.stl" scale="1 1 1" />
         </geometry>
         <material name="axis_white">
@@ -47,17 +47,26 @@
       <child link="${prefix}_base_link" />
     </joint>
-    <link name="${prefix}_camera_link" />
+    <link name="${prefix}_link" />
     <joint name="${prefix}_camera_joint" type="fixed">
       <parent link="${prefix}_base_link" />
-      <child link="${prefix}_camera_link" />
+      <child link="${prefix}_link" />
       <origin xyz="0.047 0 ${stand_height + 0.09 + 0.047}" rpy="0 0.7854 0" />
     </joint>
-    <gazebo reference="${prefix}_camera_link">
-      <material>Gazebo/Black</material>
-      <sensor type="camera" name="${prefix}_dome_camera">
+    <!--
+      Simulation support: sensor plugin
+    -->
+    <gazebo reference="${prefix}_link">
+      <plugin filename="libgz-sim-sensors-system.so" name="gz::sim::systems::Sensors">
+        <render_engine>ogre2</render_engine>
+      </plugin>
+      <sensor name="${prefix}_camera" type="camera">
         <update_rate>15</update_rate>
+        <visualize>true</visualize>
+        <always_on>true</always_on>
+        <gz_frame_id>${prefix}_link</gz_frame_id>
+        <topic>$(arg namespace)/sensors/${prefix}/image</topic>
         <camera>
-          <horizontal_fov>6.28</horizontal_fov>
-          <vertical_fov>1.57</vertical_fov>
+          <horizontal_fov>1.5184351666666667</horizontal_fov>
+          <vertical_fov>1.0122901111111111</vertical_fov>
           <image>
             <width>640</width>
@@ -66,15 +75,8 @@
           </image>
           <clip>
-            <near>0.05</near>
-            <far>500.0</far>
+            <near>0.1</near>
+            <far>100</far>
           </clip>
         </camera>
-        <plugin name="${prefix}_camera_controller" filename="libgazebo_ros_camera.so">
-          <alwaysOn>true</alwaysOn>
-          <cameraName>${prefix}_camera</cameraName>
-          <imageTopicName>${topic}</imageTopicName>
-          <cameraInfoTopicName>camera_info</cameraInfoTopicName>
-          <frameName>${prefix}_camera_link</frameName>
-        </plugin>
       </sensor>
     </gazebo>

File: clearpath_sensors_description/urdf/axis/axis_dome_ptz.urdf.xacro (robot description, xacro)
@@ -13,5 +13,5 @@
       <visual>
         <geometry>
-          <mesh filename="package://clearpath_sensors_description/meshes/axis_dome.stl" scale="1 1 1" />
+          <mesh filename="package://axis_description/meshes/axis_dome.stl" scale="1 1 1" />
         </geometry>
         <material name="axis_white">
@@ -86,35 +86,36 @@
       Add the gazebo reference frame
     -->
-    <link name="${prefix}_camera_link" />
+    <link name="${prefix}_link" />
     <joint name="${prefix}_camera_joint" type="fixed">
       <parent link="${prefix}_head_link" />
-      <child link="${prefix}_camera_link" />
+      <child link="${prefix}_link" />
       <origin xyz="0.067 0 0" rpy="0 0 0" />
     </joint>
     <!--
-      Simulation support: camera plugin & transmissions to allow control over the joints
+      Simulation support: sensor and joint controller plugins
+      Velocity control is limited to the real-world camera's limits
     -->
-    <transmission name="${prefix}_pan_trans">
-      <type>transmission_interface/SimpleTransmission</type>
-      <joint name="${prefix}_pan_joint">
-        <hardwareInterface>hardware_interface/VelocityJointInterface</hardwareInterface>
-      </joint>
-      <actuator name="${prefix}_pan_actuator">
-          <mechanicalReduction>1</mechanicalReduction>
-      </actuator>
-    </transmission>
-    <transmission name="${prefix}_tilt_trans">
-      <type>transmission_interface/SimpleTransmission</type>
-      <joint name="${prefix}_tilt_joint">
-        <hardwareInterface>hardware_interface/VelocityJointInterface</hardwareInterface>
-      </joint>
-      <actuator name="${prefix}_tilt_actuator">
-          <mechanicalReduction>1</mechanicalReduction>
-      </actuator>
-    </transmission>
-    <gazebo reference="${prefix}_camera_link">
+    <gazebo>
+      <plugin filename="libgz-sim-joint-controller-system.so" name="gz::sim::systems::JointController">
+        <joint_name>${prefix}_pan_joint</joint_name>
+        <cmd_min>-2.61</cmd_min>
+        <cmd_max>2.61</cmd_max>
+        <topic>$(arg namespace)/sensors/${prefix}/cmd_pan_vel</topic>
+      </plugin>
+      <plugin filename="libgz-sim-joint-controller-system.so" name="gz::sim::systems::JointController">
+        <joint_name>${prefix}_tilt_joint</joint_name>
+        <cmd_min>2.61</cmd_min>
+        <cmd_max>2.61</cmd_max>
+        <topic>$(arg namespace)/sensors/${prefix}/cmd_tilt_vel</topic>
+      </plugin>
+    </gazebo>
+    <gazebo reference="${prefix}_link">
       <material>Gazebo/Black</material>
-      <sensor type="camera" name="${prefix}_ptz_camera">
+      <sensor name="${prefix}_camera" type="camera">
         <update_rate>15</update_rate>
+        <visualize>true</visualize>
+        <always_on>true</always_on>
+        <gz_frame_id>${prefix}_link</gz_frame_id>
+        <topic>$(arg namespace)/sensors/${prefix}/image</topic>
         <camera>
           <horizontal_fov>1.5184351666666667</horizontal_fov>
@@ -126,15 +127,8 @@
           </image>
           <clip>
-            <near>0.05</near>
-            <far>500.0</far>
+            <near>0.1</near>
+            <far>100</far>
           </clip>
         </camera>
-        <plugin name="${prefix}_camera_controller" filename="libgazebo_ros_camera.so">
-          <alwaysOn>true</alwaysOn>
-          <cameraName>${prefix}_camera</cameraName>
-          <imageTopicName>${topic}</imageTopicName>
-          <cameraInfoTopicName>camera_info</cameraInfoTopicName>
-          <frameName>${prefix}_camera_link</frameName>
-        </plugin>
       </sensor>
     </gazebo>

File: clearpath_sensors_description/urdf/axis/axis_q62.urdf.xacro (robot description, xacro)
@@ -1,5 +1,5 @@
 <?xml version="1.0" ?>
 <robot xmlns:xacro="http://wiki.ros.org/xacro">
-  <xacro:macro name="axis_q62" params="prefix parent topic *origin">
+  <xacro:macro name="axis_q62" params="prefix parent *origin">
     <link name="${prefix}_base_link">
       <inertial>
@@ -28,5 +28,5 @@
       <visual>
         <geometry>
-          <mesh filename="package://clearpath_sensors_description/meshes/axis_q62_base.stl" scale="0.001 0.001 0.001" />
+          <mesh filename="package://axis_description/meshes/axis_q62_base.stl" scale="0.001 0.001 0.001" />
         </geometry>
         <material name="axis_grey">
@@ -62,5 +62,5 @@
       <visual>
         <geometry>
-          <mesh filename="package://clearpath_sensors_description/meshes/axis_q62_top.stl" scale="0.001 0.001 0.001" />
+          <mesh filename="package://axis_description/meshes/axis_q62_top.stl" scale="0.001 0.001 0.001" />
         </geometry>
         <material name="axis_grey">
@@ -89,5 +89,5 @@
       Add the shades & gazebo reference frame
     -->
-    <link name="${prefix}_camera_link">
+    <link name="${prefix}_link">
       <visual>
         <geometry>
@@ -95,7 +95,5 @@
         </geometry>
         <origin xyz="-0.01 0 0.05" rpy="0 0 0" />
-        <material name="axis_black">
-          <color rgba="0 0 0 1" />
-        </material>
+        <material name="black" />
       </visual>
       <visual>
@@ -104,39 +102,48 @@
         </geometry>
         <origin xyz="-0.01 0.20 0.05" rpy="0 0 0" />
-        <material name="axis_black">
-          <color rgba="0 0 0 1" />
-        </material>
+        <material name="black" />
       </visual>
+      <inertial>
+        <origin xyz="0 0 0" rpy="0 0 0" />
+        <mass value="1" />
+        <inertia
+          ixx="1.0" ixy="0.0" ixz="0.0"
+          iyy="1.0" iyz="0.0"
+          izz="1.0" />
+      </inertial>
     </link>
     <joint name="${prefix}_camera_joint" type="fixed">
       <parent link="${prefix}_head_link" />
-      <child link="${prefix}_camera_link" />
+      <child link="${prefix}_link" />
       <origin xyz="0.1 -0.107 0" rpy="0 0 0" />
     </joint>
     <!--
-      Simulation support: camera plugin & transmissions to allow control over the joints
+      Simulation support: sensor and joint controller plugins
+      Velocity control is limited to the real-world camera's limits
     -->
-    <transmission name="${prefix}_pan_trans">
-      <type>transmission_interface/SimpleTransmission</type>
-      <joint name="${prefix}_pan_joint">
-        <hardwareInterface>hardware_interface/VelocityJointInterface</hardwareInterface>
-      </joint>
-      <actuator name="${prefix}_pan_actuator">
-          <mechanicalReduction>1</mechanicalReduction>
-      </actuator>
-    </transmission>
-    <transmission name="${prefix}_tilt_trans">
-      <type>transmission_interface/SimpleTransmission</type>
-      <joint name="${prefix}_tilt_joint">
-        <hardwareInterface>hardware_interface/VelocityJointInterface</hardwareInterface>
-      </joint>
-      <actuator name="${prefix}_tilt_actuator">
-          <mechanicalReduction>1</mechanicalReduction>
-      </actuator>
-    </transmission>
-    <gazebo reference="${prefix}_camera_link">
-      <material>Gazebo/Black</material>
-      <sensor type="camera" name="${prefix}_ptz_camera">
+    <gazebo>
+      <plugin filename="libgz-sim-joint-controller-system.so" name="gz::sim::systems::JointController">
+        <joint_name>${prefix}_pan_joint</joint_name>
+        <cmd_min>-2.61</cmd_min>
+        <cmd_max>2.61</cmd_max>
+        <topic>$(arg namespace)/sensors/${prefix}/cmd_pan_vel</topic>
+      </plugin>
+      <plugin filename="libgz-sim-joint-controller-system.so" name="gz::sim::systems::JointController">
+        <joint_name>${prefix}_tilt_joint</joint_name>
+        <cmd_min>2.61</cmd_min>
+        <cmd_max>2.61</cmd_max>
+        <topic>$(arg namespace)/sensors/${prefix}/cmd_tilt_vel</topic>
+      </plugin>
+    </gazebo>
+    <gazebo reference="${prefix}_link">
+      <plugin filename="libgz-sim-sensors-system.so" name="gz::sim::systems::Sensors">
+        <render_engine>ogre2</render_engine>
+      </plugin>
+      <sensor name="${prefix}_camera" type="camera">
         <update_rate>15</update_rate>
+        <visualize>true</visualize>
+        <always_on>true</always_on>
+        <gz_frame_id>${prefix}_link</gz_frame_id>
+        <topic>$(arg namespace)/sensors/${prefix}/image</topic>
         <camera>
           <horizontal_fov>1.5184351666666667</horizontal_fov>
@@ -148,15 +155,8 @@
           </image>
           <clip>
-            <near>0.05</near>
-            <far>500.0</far>
+            <near>0.1</near>
+            <far>100</far>
           </clip>
         </camera>
-        <plugin name="${prefix}_camera_controller" filename="libgazebo_ros_camera.so">
-          <alwaysOn>true</alwaysOn>
-          <cameraName>${prefix}_camera</cameraName>
-          <imageTopicName>${topic}</imageTopicName>
-          <cameraInfoTopicName>camera_info</cameraInfoTopicName>
-          <frameName>${prefix}_camera_link</frameName>
-        </plugin>
       </sensor>
     </gazebo>

File: clearpath_sensors_description/urdf/axis_camera.urdf.xacro (robot description, xacro)
@@ -1,7 +1,4 @@
 <?xml version="1.0" ?>
 <robot xmlns:xacro="http://www.ros.org/wiki/xacro">
-    <xacro:include filename="$(find clearpath_sensors_description)/urdf/axis/axis_dome_fixed.urdf.xacro"/>
-    <xacro:include filename="$(find clearpath_sensors_description)/urdf/axis/axis_dome_ptz.urdf.xacro"/>
-    <xacro:include filename="$(find clearpath_sensors_description)/urdf/axis/axis_q62.urdf.xacro"/>
     <xacro:macro name="axis_camera" params="
         name
@@ -9,12 +6,12 @@
         *origin
         model:=dome_ptz
-        topic:=image_raw
+        topic:=image
         update_rate:=15
     ">
         <xacro:if value="${model == 'dome_fixed'}">
+            <xacro:include filename="$(find clearpath_sensors_description)/urdf/axis/axis_dome_fixed.urdf.xacro"/>
             <xacro:axis_dome_fixed
                 prefix="${name}"
                 parent="${parent_link}"
-                topic="${topic}"
             >
                 <xacro:insert_block name="origin" />
@@ -22,8 +19,8 @@
         </xacro:if>
         <xacro:if value="${model == 'dome_ptz'}">
+            <xacro:include filename="$(find clearpath_sensors_description)/urdf/axis/axis_dome_ptz.urdf.xacro"/>
             <xacro:axis_dome_ptz
                 prefix="${name}"
                 parent="${parent_link}"
-                topic="${topic}"
             >
                 <xacro:insert_block name="origin" />
@@ -31,8 +28,8 @@
         </xacro:if>
         <xacro:if value="${model == 'q62'}">
+            <xacro:include filename="$(find clearpath_sensors_description)/urdf/axis/axis_q62.urdf.xacro"/>
             <xacro:axis_q62
                 prefix="${name}"
                 parent="${parent_link}"
-                topic="${topic}"
             >
                 <xacro:insert_block name="origin" />
