Commit message: Add plugins to get the PTZ joint states out of gazebo and into ROS (#126)

File: clearpath_sensors_description/urdf/axis/axis_dome_ptz.urdf.xacro (robot description, xacro)
@@ -109,4 +109,12 @@
         <topic>$(arg namespace)/sensors/${prefix}/cmd_tilt_vel</topic>
       </plugin>
+      <plugin filename="gz-sim-joint-state-publisher-system" name="gz::sim::systems::JointStatePublisher">
+        <joint_name>${prefix}_pan_joint</joint_name>
+        <topic>$(arg namespace)/sensors/${prefix}/pan_joint_state</topic>
+      </plugin>
+      <plugin filename="gz-sim-joint-state-publisher-system" name="gz::sim::systems::JointStatePublisher">
+        <joint_name>${prefix}_tilt_joint</joint_name>
+        <topic>$(arg namespace)/sensors/${prefix}/tilt_joint_state</topic>
+      </plugin>
     </gazebo>
     <gazebo reference="${prefix}_link">

File: clearpath_sensors_description/urdf/axis/axis_q62.urdf.xacro (robot description, xacro)
@@ -95,5 +95,7 @@
         </geometry>
         <origin xyz="-0.01 0 0.05" rpy="0 0 0" />
-        <material name="black" />
+        <material name="black">
+          <color rgba="0 0 0 1" />
+        </material>
       </visual>
       <visual>
@@ -102,5 +104,7 @@
         </geometry>
         <origin xyz="-0.01 0.20 0.05" rpy="0 0 0" />
-        <material name="black" />
+        <material name="black">
+          <color rgba="0 0 0 1" />
+        </material>
       </visual>
       <inertial>
@@ -135,4 +139,12 @@
         <topic>$(arg namespace)/sensors/${prefix}/cmd_tilt_vel</topic>
       </plugin>
+      <plugin filename="gz-sim-joint-state-publisher-system" name="gz::sim::systems::JointStatePublisher">
+        <joint_name>${prefix}_pan_joint</joint_name>
+        <topic>$(arg namespace)/sensors/${prefix}/pan_joint_state</topic>
+      </plugin>
+      <plugin filename="gz-sim-joint-state-publisher-system" name="gz::sim::systems::JointStatePublisher">
+        <joint_name>${prefix}_tilt_joint</joint_name>
+        <topic>$(arg namespace)/sensors/${prefix}/tilt_joint_state</topic>
+      </plugin>
     </gazebo>
     <gazebo reference="${prefix}_link">
