Commit message: Fix test errors (#132)
* Add continue clause to the unsupported device/platform exceptions so we don't try any further tests with them

* Fix URDF parameters so the source CI passes with the axis cameras

File: clearpath_sensors_description/urdf/axis/axis_dome_fixed.urdf.xacro (robot description, xacro)
@@ -1,5 +1,5 @@
 <?xml version="1.0" ?>
 <robot xmlns:xacro="http://wiki.ros.org/xacro">
-  <xacro:macro name="axis_dome_fixed" params="prefix parent topic stand_height:=0.062 *origin">
+  <xacro:macro name="axis_dome_fixed" params="prefix parent stand_height:=0.062 *origin">
     <link name="${prefix}_base_link">
       <inertial>

File: clearpath_sensors_description/urdf/axis/axis_dome_ptz.urdf.xacro (robot description, xacro)
@@ -1,5 +1,5 @@
 <?xml version="1.0" ?>
 <robot xmlns:xacro="http://wiki.ros.org/xacro">
-  <xacro:macro name="axis_dome_ptz" params="prefix parent topic stand_height:=0.062 *origin">
+  <xacro:macro name="axis_dome_ptz" params="prefix parent stand_height:=0.062 *origin">
     <link name="${prefix}_base_link">
       <inertial>
